File: eagle/house-sensor4pre.brd (EAGLE design)
At the start: 95.6 x 72.4 mm, 72 parts, among them Q1 C1815, Q2 C1815, Q3 C1815, T1 NJL7502L, U1 MCP3208/D, U2 NJU7072D

Commit message: change some constant
Parts:
- C11, C12: value .1uF -> 1u
- L1, L2: value 47uH -> 47u
- R1, R7: value 2.2k -> 1k
- R28, R30: value 100k -> 10k
Changed lines of the file:
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@@
 </element>
 <element name="R3" library="akihabara" package="0207/2V" value="1k±1%" x="27.94" y="48.895" rot="R180"/>
-<element name="R1" library="akihabara" package="0207/2V" value="2.2k" x="9.525" y="50.165" rot="R270"/>
+<element name="R1" library="akihabara" package="0207/2V" value="1k" x="9.525" y="50.165" rot="R270"/>
 <element name="R5" library="akihabara" package="0207/2V" value="1k±1%" x="6.985" y="55.88" rot="R90"/>
 <element name="R6" library="akihabara" package="0207/2V" value="10k±1%" x="11.43" y="58.42" rot="R90"/>
@@
 <attribute name="OC_FARNELL" value="unknown" x="-28.575" y="48.895" size="1.778" layer="27" rot="R270" display="off"/>
 </element>
-<element name="R7" library="akihabara" package="0207/2V" value="2.2k" x="38.735" y="53.34" rot="R90"/>
+<element name="R7" library="akihabara" package="0207/2V" value="1k" x="38.735" y="53.34" rot="R90"/>
 <element name="R8" library="akihabara" package="0204/7" value="100k" x="32.385" y="53.34" rot="R270"/>
 <element name="PIN" library="con-lstb" package="MA13-2" value="ToRpi" x="45.085" y="27.94" rot="R180">
@@
 <attribute name="OC_FARNELL" value="unknown" x="41.275" y="66.675" size="1.778" layer="27" rot="R270" display="off"/>
 </element>
-<element name="R28" library="akihabara" package="0204V" value="100k" x="45.085" y="50.165" rot="R270"/>
-<element name="C11" library="akihabara" package="C050-024X044" value=".1uF" x="31.75" y="43.815"/>
+<element name="R28" library="akihabara" package="0204V" value="10k" x="45.085" y="50.165" rot="R270"/>
+<element name="C11" library="akihabara" package="C050-024X044" value="1u" x="31.75" y="43.815"/>
 <element name="PILOT" library="eagle-ltspice" package="LED_LD260" value="LED" x="86.36" y="17.145" rot="R90">
 <attribute name="SPICEMODEL" value="NONE" x="86.36" y="17.145" size="1.778" layer="27" rot="R90" display="off"/>
@@
 </element>
 <element name="R14" library="akihabara" package="0204V" value="1k" x="42.545" y="33.655" rot="R90"/>
-<element name="L1" library="inductors" package="LBC-SE" value="47uH" x="45.085" y="55.88" rot="R270"/>
+<element name="L1" library="inductors" package="LBC-SE" value="47u" x="45.085" y="55.88" rot="R270"/>
 <element name="R29" library="akihabara" package="0207/5V" value="1k" x="45.085" y="64.135" rot="R270"/>
 <element name="D2" library="1-diode" package="DIODE_V" value="Schottky" x="10.16" y="35.56" rot="R180"/>
@@
 <attribute name="OC_FARNELL" value="unknown" x="59.055" y="66.675" size="1.778" layer="27" rot="R270" display="off"/>
 </element>
-<element name="R30" library="akihabara" package="0204V" value="100k" x="53.34" y="50.165" rot="R270"/>
-<element name="C12" library="akihabara" package="C050-024X044" value=".1uF" x="31.75" y="38.735"/>
-<element name="L2" library="inductors" package="LBC-SE" value="47uH" x="53.34" y="55.88" rot="R270"/>
+<element name="R30" library="akihabara" package="0204V" value="10k" x="53.34" y="50.165" rot="R270"/>
+<element name="C12" library="akihabara" package="C050-024X044" value="1u" x="31.75" y="38.735"/>
+<element name="L2" library="inductors" package="LBC-SE" value="47u" x="53.34" y="55.88" rot="R270"/>
 <element name="R31" library="akihabara" package="0207/5V" value="1k" x="53.34" y="64.135" rot="R270"/>
 <element name="LUX1" library="con-lstb" package="MA03-1" value="LUX" x="15.24" y="66.675" rot="R270">
