File: eagle/house-sensor4pre.sch (EAGLE design)
At the start: 72 parts, among them Q1 C1815, Q2 C1815, Q3 C1815, T1 NJL7502L, U1 MCP3208/D, U2 NJU7072D

Commit message: change some constant
Parts:
- C11, C12: value .1uF -> 1u
- L1, L2: value 47uH -> 47u
- R1, R7: value 2.2k -> 1k
- R28, R30: value 100k -> 10k
Other:
- note removed: "fc=33Hz"
Changed lines of the file:
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@@
 <part name="T1" library="opto-trans-siemens" deviceset="BPX81" device="" value="NJL7502L"/>
 <part name="R3" library="akihabara" deviceset="R-US_" device="0207/2V" value="1k±1%"/>
-<part name="R1" library="akihabara" deviceset="R-US_" device="0207/2V" value="2.2k"/>
+<part name="R1" library="akihabara" deviceset="R-US_" device="0207/2V" value="1k"/>
 <part name="R5" library="akihabara" deviceset="R-US_" device="0207/2V" value="1k±1%"/>
 <part name="R6" library="akihabara" deviceset="R-US_" device="0207/2V" value="10k±1%"/>
@@
 <part name="+3V1" library="supply1" deviceset="+3V3" device=""/>
 <part name="LUX2" library="con-lstb" deviceset="MA03-1" device="" value="LUX"/>
-<part name="R7" library="akihabara" deviceset="R-US_" device="0207/2V" value="2.2k"/>
+<part name="R7" library="akihabara" deviceset="R-US_" device="0207/2V" value="1k"/>
 <part name="R8" library="akihabara" deviceset="R-US_" device="0204/7" value="100k"/>
 <part name="+3V5" library="supply1" deviceset="+3V3" device=""/>
@@
 <part name="SUPPLY23" library="supply2" deviceset="GND" device=""/>
 <part name="+3V11" library="supply1" deviceset="+3V3" device=""/>
-<part name="R28" library="akihabara" deviceset="R-US_" device="0204/2V" value="100k"/>
-<part name="C11" library="akihabara" deviceset="C-EU" device="050-024X044" value=".1uF"/>
+<part name="R28" library="akihabara" deviceset="R-US_" device="0204/2V" value="10k"/>
+<part name="C11" library="akihabara" deviceset="C-EU" device="050-024X044" value="1u"/>
 <part name="SUPPLY24" library="supply2" deviceset="GND" device=""/>
 <part name="PILOT" library="eagle-ltspice" deviceset="LED_E" device="LD260" value="LED"/>
 <part name="R14" library="akihabara" deviceset="R-US_" device="0204/2V" value="1k"/>
 <part name="SUPPLY27" library="supply2" deviceset="GND" device=""/>
-<part name="L1" library="inductors" deviceset="LBC-SE" device="" value="47uH"/>
+<part name="L1" library="inductors" deviceset="LBC-SE" device="" value="47u"/>
 <part name="R29" library="akihabara" deviceset="R-US_" device="0207/5V" value="1k"/>
 <part name="D2" library="1-diode" deviceset="DIODE_V" device="" value="Schottky"/>
@@
 <part name="SUPPLY25" library="supply2" deviceset="GND" device=""/>
 <part name="+3V12" library="supply1" deviceset="+3V3" device=""/>
-<part name="R30" library="akihabara" deviceset="R-US_" device="0204/2V" value="100k"/>
-<part name="C12" library="akihabara" deviceset="C-EU" device="050-024X044" value=".1uF"/>
+<part name="R30" library="akihabara" deviceset="R-US_" device="0204/2V" value="10k"/>
+<part name="C12" library="akihabara" deviceset="C-EU" device="050-024X044" value="1u"/>
 <part name="SUPPLY26" library="supply2" deviceset="GND" device=""/>
-<part name="L2" library="inductors" deviceset="LBC-SE" device="" value="47uH"/>
+<part name="L2" library="inductors" deviceset="LBC-SE" device="" value="47u"/>
 <part name="R31" library="akihabara" deviceset="R-US_" device="0207/5V" value="1k"/>
 <part name="+3V13" library="supply1" deviceset="+3V3" device=""/>
@@
 <sheet>
 <plain>
-<text x="27.94" y="-224.79" size="1.778" layer="91">fc=33Hz</text>
 <text x="-5.08" y="77.47" size="1.778" layer="91" align="bottom-right">NJL7502L C
 NJL7502L E
